File: electronics/rev2/rc-winch-controller.kicad_pcb (KiCad board)
At the start: 2 copper layers, 31 x 17 mm, 14 parts, among them J1 Conn_01x06, J2 Conn_01x06, SW1 SETUP, U1 MCP1703A-3302_SOT23, U2 LPC812M001JDH16, U3 RZ7889

Commit message: Update PCB
Parts:
- removed C4: CP, Capacitor_THT:CP_Axial_L11.0mm_D6.0mm_P18.00mm_Horizontal
- C1, C2: footprint Capacitor_SMD:C_0805_2012Metric_Pad1.18x1.45mm_HandSolder -> Capacitor_SMD:C_0805_2012Metric
- C3: footprint Capacitor_SMD:C_0603_1608Metric_Pad1.08x0.95mm_HandSolder -> Capacitor_SMD:C_0603_1608Metric
- D1: footprint Package_TO_SOT_SMD:SOT-523 -> Package_TO_SOT_SMD:SOT-23
- U1: footprint Package_TO_SOT_SMD:SOT-23_Handsoldering -> Package_TO_SOT_SMD:SOT-23W
- moved J1 56.2 mm to (128.0, 98.5)
- moved D2 47.5 mm to (123.6, 96.4), turned to 90 degrees
- moved RN1 47.5 mm to (123.9, 91.4), turned to 180 degrees
- moved D1 36.5 mm to (122.4, 86.8)
- moved U2 36.0 mm to (118.3, 96.4), turned to 180 degrees
- moved SW1 36.0 mm to (114.2, 91.0), turned to 0 degrees
- moved C2 32.1 mm to (111.9, 86.8)
- moved C3 31.6 mm to (113.2, 95.8), turned to 270 degrees
- moved U1 29.2 mm to (115.5, 86.8)
- moved C1 28.1 mm to (119.0, 86.8), turned to 90 degrees
- moved U3 17.7 mm to (108.3, 96.8), turned to 180 degrees
- moved F1 16.1 mm to (106.6, 90.3), turned to 270 degrees
- moved J2 5.91 mm to (102.0, 98.5)
Connections:
- J1 pad 3: /ST-Rx-in -> /AUX-Rx-in
- J1 pad 5: (no net) -> GND
- J1 pad 6: (no net) -> /VMOT
- J2 pad 1: /MOT1 -> /MOT2
- J2 pad 2: /MOT2 -> /MOT1
- RN1 pad 1: /Tx-in -> /LED-A
- RN1 pad 3: /LED-A -> /AUX-Rx-in
- RN1 pad 4: /ST-Rx-in -> /Tx-in
- RN1 pad 5: /ST-Rx -> /Tx
- RN1 pad 6: /VDD -> /AUX-Rx
- RN1 pad 8: /Tx -> /VDD
- U2 pad 1: (no net) -> /LED-R
- U2 pad 16: /ST-Rx -> /AUX-Rx
- U2 pad 5: /LED-R -> /LED-G
- U2 pad 6: /LED-G -> /LED-B
- U2 pad 9: /LED-B -> (no net)
Routing:
- net /AUX-Rx: track 0.00 -> 18.4 mm
- net /VIN: track 35.9 -> 48.9 mm, vias 2 -> 5
- net /VMOT: track 18.9 -> 29.6 mm, vias 2 -> 0
- net GND: track 6.36 -> 16.9 mm, vias 1 -> 8
- net /ST-Rx: track 8.30 -> 0.00 mm
- net /LED-B: track 9.47 -> 2.07 mm
- net /VDD: track 18.5 -> 23.5 mm, vias 2 -> 3
- net /AUX-Rx-in: track 0.00 -> 4.66 mm
- net /SW-ISP: track 13.4 -> 9.35 mm, vias 2 -> 0
- net /ST-Rx-in: track 3.61 -> 0.00 mm
- net /LED-A: track 4.99 -> 7.77 mm
- net /Tx: track 8.93 -> 11.1 mm, vias 2 -> 0
- net /FWD: track 3.22 -> 4.97 mm
- net Net-(C1-Pad1): track 7.76 -> 6.07 mm
- net /REV: track 3.37 -> 4.71 mm
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Other:
- board size 31 x 17 mm -> 30 x 16 mm
- net class Default: clearance 0.2 -> 0.2032; trace_width 0.25 -> 0.254
- rule trace_clearance: 0.2 -> 0.2032
- rule trace_min: 0.2 -> 0.2032
- board text added: "+"
- board text added: "+Motor"
- board text added: "-"
- board text added: "4..13V"
- board text added: "AUX/SW/Rx"
- board text added: "C"
- board text added: "LANE Boys RC"
- board text added: "RC Winch Controller"
- board text added: "SW/Tx"
- board text added: "Winch1"
- board text added: "Winch2"
